File: kicad/pcb-custom.sch (KiCad schematic (older format))
At the start: 37 parts, among them J1 Conn_VIN, J2 Conn_02x07_Odd_Even, J3 Conn_3V3, J4 Conn_PortB, J5 Conn_PortA, SW1 SW_Push, U1 AMS1117-3.3, U2 STM32L452CEU6

Commit message: Start routing
Parts:
- added C14, C15: 100 nF, Capacitor_SMD:C_0402_1005Metric, symbol Device:C_Small
- added SW2, SW3: SW_Push, Button_Switch_SMD:SW_SPST_EVQP0, symbol Switch:SW_Push
- C1, C11, C12: footprint (none) -> Capacitor_SMD:C_0805_2012Metric
- C10, C13, C2, C3, C4, C5, C6, C7, C8, C9: footprint (none) -> Capacitor_SMD:C_0402_1005Metric
- D1: footprint (none) -> Diode_SMD:D_SOD-123
- D2, D3, D4, D5: footprint (none) -> LED_SMD:LED_0603_1608Metric
- F1: footprint (none) -> Fuse:Fuse_0603_1608Metric
- FB1, FB2: footprint (none) -> Inductor_SMD:L_0805_2012Metric
- H1, H2, H3, H4: footprint (none) -> MountingHole:MountingHole_4.3mm_M4_Pad_Via
- J1, J3: footprint (none) -> Connector_PinHeader_2.54mm:PinHeader_1x02_P2.54mm_Vertical
- J2: footprint (none) -> Connector_PinHeader_1.27mm:PinHeader_2x07_P1.27mm_Vertical
- J4, J5: footprint (none) -> Connector_PinHeader_2.54mm:PinHeader_1x16_P2.54mm_Vertical
- R1, R2, R3, R4: footprint (none) -> Resistor_SMD:R_0603_1608Metric
- SW1: footprint (none) -> Button_Switch_SMD:SW_SPST_EVQP0
Connections:
- net GND: now also C14.2, C15.2, SW2.1, SW3.1
- net BTN1: now reaches J4.1 (Pin_1), U2.18 (PB0)
- net BTN1: now also C14.1, SW2.2
- net BTN2: now reaches J4.2 (Pin_2), U2.19 (PB1)
- net BTN2: now also C15.1, SW3.2
