File: kicad/pcb-custom.kicad_pcb (KiCad board)
At the start: 4 copper layers, 70 x 70 mm, 41 parts, among them J1 Conn_VIN, J2 Conn_02x07_Odd_Even, J3 Conn_3V3, J4 Conn_PortB, J5 Conn_PortA, SW1 SW_Push, SW2 SW_Push, SW3 SW_Push, U1 AMS1117-3.3, U2 STM32L452CEU6

Commit message: Complete routing
Parts:
- moved C6 1.33 mm to (81.3, 52.3)
- moved C7 1.33 mm to (82.3, 52.3)
- moved C10 0.90 mm to (73.9, 49.1)
- moved C9 0.90 mm to (73.9, 48.1)
- moved C4 0.51 mm to (78.0, 59.9)
- moved C8 0.51 mm to (78.0, 60.9)
Routing:
- net SWCLK: track 0.00 -> 134.2 mm
- net SWDIO: track 0.00 -> 121.4 mm, vias 0 -> 1
- net BTN2: track 34.2 -> 134.5 mm, vias 0 -> 1
- net BTN1: track 34.6 -> 123.0 mm
- net Net-(J4-Pad5): track 0.00 -> 87.0 mm, vias 0 -> 1
- net LED_GREEN: track 0.00 -> 86.0 mm, vias 0 -> 4
- net LED_BLUE: track 0.00 -> 85.7 mm, vias 0 -> 4
- net Net-(J4-Pad6): track 0.00 -> 82.4 mm, vias 0 -> 1
- net Net-(J5-Pad9): track 0.00 -> 80.7 mm, vias 0 -> 1
- net Net-(J4-Pad7): track 0.00 -> 79.0 mm, vias 0 -> 1
- net Net-(J4-Pad8): track 0.00 -> 75.5 mm, vias 0 -> 1
- net NRST: track 27.5 -> 100.4 mm, vias 2 -> 3
- net Net-(J4-Pad9): track 0.00 -> 72.6 mm, vias 0 -> 1
- net Net-(J5-Pad10): track 0.00 -> 72.2 mm, vias 0 -> 1
- net Net-(J4-Pad10): track 0.00 -> 69.7 mm, vias 0 -> 1
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Other:
- board text added: "+"
- board text added: "+3V3"
- board text added: "1"
- board text added: "2"
- board text added: "BTN1"
- board text added: "BTN2"
- board text added: "GND"
- board text added: "LED1"
- board text added: "LED2"
- board text added: "LED3"
- board text added: "PA0"
- board text added: "PA1"
- board text added: "PA10"
- board text added: "PA11"
- board text added: "PA12"
- board text added: "PA13"
- board text added: "PA14"
- board text added: "PA15"
- board text added: "PA2"
- board text added: "PA3"
- board text added: "PA4"
- board text added: "PA5"
- board text added: "PA6"
- board text added: "PA7"
- board text added: "PA8"
- board text added: "PA9"
- board text added: "PB0"
- board text added: "PB1"
- board text added: "PB10"
- board text added: "PB11"
- board text added: "PB12"
- board text added: "PB13"
- board text added: "PB14"
- board text added: "PB15"
- board text added: "PB2"
- board text added: "PB3"
- board text added: "PB4"
- board text added: "PB5"
- board text added: "PB6"
- board text added: "PB7"
- board text added: "PB8"
- board text added: "PB9"
- board text added: "PORT A"
- board text added: "PORT B"
- board text added: "RST"
- board text added: "STLINK"
- board text added: "VCC"
- board text added: "VIN"
- board text added: "by @ayoubsabri & @kokkonisd july 2020"
- board text added: "walk it like I talk it"
